File: docs/proyecto/memoria/fig/diagramas_FPGA/diagramas_funcionamiento/diagramas_funcionamiento.sch (KiCad schematic (older format))
At the start: 12 parts

Commit message: Esquemas FPGA
Parts:
- U: renamed from U?; DIVIDER DIVIDER = 24 -> (none)
- U?: DIVIDER DIVIDER = 24 -> (none)
- U?: DIVIDER DIVIDER = 19 -> (none)
- U?: Baudrate 3750000bauds -> (none)
Connections:
- net labels added: 19, 24, 3750000
- wire segments 185 -> 198
Other:
- note added: "FPGA ICE40HX1K"
